File: 1_Circuito/1_Transmisor/2_CIRCUITS/1_CARACTERIZACION_LED/shield_arduino/shield_arduino.kicad_pcb (KiCad board)
At the start: 2 copper layers, 53.8 x 98.7 mm, 21 parts, among them J1 QWIIC_5v, J2 LED ext, J3 LCD NOKIA 5110, J4 QWIIC_5v, Q1 2N3904, SW1 RESET, U1 LM358

Commit message: feat: export KiCad PCB fabrication files and update characterization LED project documentation
Connections:
- A1 pad 5V1: +5V -> unconnected-(A1-5V-Pad5V1)
- A1 pad GND2: GND -> GND2
- A1 pad GND4: GND -> GND1
- J3 pad 7: GND -> GND1
- J3 pad 8: GND -> GND1
- R5 pad 2: GND -> GND2
- RV1 pad 3: GND -> GND2
Routing:
- net GND: track 169.4 -> 79.6 mm
- net GND2: track 0.00 -> 59.5 mm
- net GND1: track 0.00 -> 36.8 mm
- net Net-(A1-RESET): track 45.0 -> 51.5 mm
