File: 1_Circuito/1_Transmisor/2_CIRCUITS/1_CARACTERIZACION_LED/shield_arduino/shield_arduino.kicad_sch (KiCad schematic)
At the start: 21 parts, among them J1 QWIIC_5v, J2 LED ext, J3 LCD NOKIA 5110, J4 QWIIC_5v, Q1 2N3904, SW1 RESET, U1 LM358

Commit message: feat: export KiCad PCB fabrication files and update characterization LED project documentation
Connections:
- net +5V: no longer A1.5V1 (5V)
- net GND: no longer A1.GND2 (GND), A1.GND4 (SPI_GND), J3.7 (Pin_7), J3.8 (Pin_8), R5.2, RV1.3
- new net GND1: A1.GND4 (SPI_GND), J3.7 (Pin_7), J3.8 (Pin_8)
- new net GND2: A1.GND2 (GND), R5.2, RV1.3

Commit message: Refactor code structure for improved readability and maintainability
Other:
- title: (none) -> Proyecto fluorimetro
Changed lines of the file:
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@@
 	(generator_version "10.0")
 	(paper "A4")
+	(title_block
+		(title "Proyecto fluorimetro")
+		(date "2026-08-31")
+	)
 	(rectangle
 		(start 180.34 55.118)
